Commit message: added lidar

File: description/robot.urdf.xacro (robot description, xacro)
@@ -3,3 +3,4 @@
     <xacro:include filename="/home/user/jerin_ws/src/my_bot/description/robot_core.xacro" />
     <xacro:include filename="/home/user/jerin_ws/src/my_bot/description/gazebo_control.xacro" />
+    <xacro:include filename="/home/user/jerin_ws/src/my_bot/description/lidar.xacro" />
 </robot>

File: description/robot_core.xacro (robot description, xacro)
@@ -13,4 +13,7 @@
     <material name="orange">
         <color rgba="1 0.3 0.1 1"/>
+    </material>
+    <material name="red">
+        <color rgba="1 0 0 1"/>
     </material>
     <link name="base_link" />
